Commit message: Started the process of making the simulator fully compliant with hardware. Still need the robot working in order to verify.

File: davinci_gazebo/model/both_psms_sticky.urdf.xacro (robot description, xacro)
@@ -59,5 +59,5 @@
 	<gazebo>
 		<plugin name="gazebo_ros_control" filename="libgazebo_ros_control.so">
-			<robotNamespace>/davinci</robotNamespace>
+			<robotNamespace>davinci</robotNamespace>
 			<robotSimType>gazebo_ros_control/DefaultRobotHWSim</robotSimType>
 		</plugin>

File: davinci_gazebo/model/gazebo_psm_sticky.tool.sca.urdf.xacro (robot description, xacro)
@@ -9,5 +9,5 @@
 	<xacro:macro name="psm_tool_sca" params="prefix">
 		<!-- joint 5: Outer wrist pitch joint -->
-		<joint name="${prefix}outer_wrist_pitch_joint" type="revolute">
+		<joint name="${prefix}outer_wrist_pitch" type="revolute">
 			<parent link="${prefix}tool_wrist_shaft_link"/>
 			<child link="${prefix}tool_wrist_sca_link"/>
@@ -42,5 +42,5 @@
 		</link>
 		<!-- joint 6: Outer wrist yaw joint -->
-		<joint name="${prefix}outer_wrist_yaw_joint" type="revolute">
+		<joint name="${prefix}outer_wrist_yaw" type="revolute">
 			<parent link="${prefix}tool_wrist_sca_link"/>
 			<child link="${prefix}tool_wrist_sca_shaft_link"/>
@@ -65,5 +65,5 @@
 		</link>
 		<!-- joint 7-1: Outer open angle 1  -->
-		<joint name="${prefix}outer_wrist_open_angle_joint" type="revolute">
+		<joint name="${prefix}jaw" type="revolute">
 			<parent link="${prefix}tool_wrist_sca_shaft_link"/>
 			<child link="${prefix}tool_wrist_sca_ee_link_1"/>
@@ -87,5 +87,5 @@
 		</link>
 		<!-- joint 7-2: Outer open angle 2   -->
-		<joint name="${prefix}outer_wrist_open_angle_joint_mimic" type="revolute">
+		<joint name="${prefix}jaw_mimic" type="revolute">
 			<parent link="${prefix}tool_wrist_sca_shaft_link"/>
 			<child link="${prefix}tool_wrist_sca_ee_link_2"/>
@@ -146,5 +146,5 @@
 		</link>
 		<!-- attach fingertip pad  -->
-		<joint name="${prefix}fingertip2_joint" type="fixed">
+		<joint name="${prefix}fingertip2" type="fixed">
 			<parent link="${prefix}tool_wrist_sca_ee_link_2"/>
 			<child link="${prefix}fingertip2"/>
@@ -189,5 +189,5 @@
 		</link>
 		<!-- attach fingertip pad 1  -->
-		<joint name="${prefix}fingertip1_joint" type="fixed">
+		<joint name="${prefix}fingertip1" type="fixed">
 			<parent link="${prefix}tool_wrist_sca_ee_link_1"/>
 			<child link="${prefix}fingertip1"/>
@@ -196,5 +196,5 @@
 		</joint>
 		<!-- tool tip -->
-		<joint name="${prefix}tool_tip_joint_" type="fixed">
+		<joint name="${prefix}tool_tip_" type="fixed">
 			<parent link="${prefix}tool_wrist_sca_shaft_link"/>
 			<child link="${prefix}tool_tip_link"/>
@@ -234,5 +234,5 @@
 		<transmission name="${prefix}tran5">
 			<type>transmission_interface/SimpleTransmission</type>
-			<joint name="${prefix}outer_wrist_pitch_joint">
+			<joint name="${prefix}outer_wrist_pitch">
 				<hardwareInterface>EffortJointInterface</hardwareInterface>
 			</joint>
@@ -244,5 +244,5 @@
 		<transmission name="${prefix}tran6">
 			<type>transmission_interface/SimpleTransmission</type>
-			<joint name="${prefix}outer_wrist_yaw_joint">
+			<joint name="${prefix}outer_wrist_yaw">
 				<hardwareInterface>EffortJointInterface</hardwareInterface>
 			</joint>
@@ -254,5 +254,5 @@
 		<transmission name="${prefix}tran7">
 			<type>transmission_interface/SimpleTransmission</type>
-			<joint name="${prefix}outer_wrist_open_angle_joint">
+			<joint name="${prefix}jaw">
 				<hardwareInterface>EffortJointInterface</hardwareInterface>
 			</joint>
@@ -264,5 +264,5 @@
 		<transmission name="${prefix}tran7_mimic">
 			<type>transmission_interface/SimpleTransmission</type>
-			<joint name="${prefix}outer_wrist_open_angle_joint_mimic">
+			<joint name="${prefix}jaw_mimic">
 				<hardwareInterface>EffortJointInterface</hardwareInterface>
 			</joint>

File: dvrk_model/model/both_psms.urdf (robot description, URDF)
Before this commit: robot dvrk_psm, 24 links, 23 joints
Joints:
- removed joint one_outer_insertion_joint
- removed joint one_outer_pitch_joint
- removed joint one_outer_pitch_joint_1
- removed joint one_outer_pitch_joint_2
- removed joint one_outer_pitch_joint_3
- removed joint one_outer_pitch_joint_4
- removed joint one_outer_pitch_joint_5
- removed joint one_outer_roll_joint
- removed joint one_outer_yaw_joint
- removed joint two_outer_insertion_joint
- removed joint two_outer_pitch_joint
- removed joint two_outer_pitch_joint_1
- removed joint two_outer_pitch_joint_2
- removed joint two_outer_pitch_joint_3
- removed joint two_outer_pitch_joint_4
- removed joint two_outer_pitch_joint_5
- removed joint two_outer_roll_joint
- removed joint two_outer_roll_shaft_joint
- removed joint two_outer_yaw_joint
- added joint one_outer_insertion: type prismatic, parent one_outer_pitch_link, child one_tool_main_link, origin xyz=0 0.4318 0 rpy=1.5708 0 0, axis 0 0 1, limit lower=0 upper=0.240 effort=1000 velocity=.4
- added joint one_outer_pitch: type revolute, parent one_outer_yaw_link, child one_outer_pitch_link, origin xyz=0 0 0 rpy=-1.5708 -1.5708 0, axis 0 0 1, limit lower=-0.7854 upper=0.7854 effort=1000 velocity=.4
- added joint one_outer_pitch_1: type continuous, parent one_outer_yaw_link, child one_outer_pitch_back_link, origin xyz=0 0.0295 0.5185 rpy=-1.5708 -1.5708 0, axis 0 0 1, mimic joint=one_outer_pitch multiplier=1
- added joint one_outer_pitch_2: type continuous, parent one_outer_yaw_link, child one_outer_pitch_front_link, origin xyz=0 0.0295 0.4285 rpy=-1.5708 -1.5708 0, axis 0 0 1, mimic joint=one_outer_pitch multiplier=1
- added joint one_outer_pitch_3: type continuous, parent one_outer_pitch_back_link, child one_outer_pitch_bottom_link, origin xyz=0.04178 0.15007 -0.0137 rpy=0 0 0, axis 0 0 1, mimic joint=one_outer_pitch multiplier=-1
- added joint one_outer_pitch_4: type continuous, parent one_outer_pitch_back_link, child one_outer_pitch_top_link, origin xyz=0.04209 0.18695 -0.02412 rpy=0 0 0, axis 0 0 1, mimic joint=one_outer_pitch multiplier=-1
- added joint one_outer_pitch_5: type continuous, parent one_outer_pitch_bottom_link, child one_outer_insertion_link, origin xyz=-0.520 0 -0.0155 rpy=0 0 0, axis 0 0 1, mimic joint=one_outer_pitch multiplier=1
- added joint one_outer_roll: type revolute, parent one_tool_main_link, child one_tool_wrist_link, origin xyz=0 0 0.4162 rpy=0 0 0, axis 0 0 1, limit lower=-2.2689 upper=2.2689 effort=1000 velocity=.4
- added joint one_outer_yaw: type revolute, parent one_psm_base_link, child one_outer_yaw_link, origin xyz=0.0 0.0 0.0 rpy=0 -1.5708 1.5708, axis 0 0 1, limit lower=-1.5707 upper=1.5707 effort=1000 velocity=.4
- added joint two_outer_insertion: type prismatic, parent two_outer_pitch_link, child two_tool_main_link, origin xyz=0 0.4318 0 rpy=1.5708 0 0, axis 0 0 1, limit lower=0 upper=0.240 effort=1000 velocity=.4
- added joint two_outer_pitch: type revolute, parent two_outer_yaw_link, child two_outer_pitch_link, origin xyz=0 0 0 rpy=-1.5708 -1.5708 0, axis 0 0 1, limit lower=-0.7854 upper=0.7854 effort=1000 velocity=.4
- added joint two_outer_pitch_1: type continuous, parent two_outer_yaw_link, child two_outer_pitch_back_link, origin xyz=0 0.0295 0.5185 rpy=-1.5708 -1.5708 0, axis 0 0 1, mimic joint=two_outer_pitch multiplier=1
- added joint two_outer_pitch_2: type continuous, parent two_outer_yaw_link, child two_outer_pitch_front_link, origin xyz=0 0.0295 0.4285 rpy=-1.5708 -1.5708 0, axis 0 0 1, mimic joint=two_outer_pitch multiplier=1
- added joint two_outer_pitch_3: type continuous, parent two_outer_pitch_back_link, child two_outer_pitch_bottom_link, origin xyz=0.04178 0.15007 -0.0137 rpy=0 0 0, axis 0 0 1, mimic joint=two_outer_pitch multiplier=-1
- added joint two_outer_pitch_4: type continuous, parent two_outer_pitch_back_link, child two_outer_pitch_top_link, origin xyz=0.04209 0.18695 -0.02412 rpy=0 0 0, axis 0 0 1, mimic joint=two_outer_pitch multiplier=-1
- added joint two_outer_pitch_5: type continuous, parent two_outer_pitch_bottom_link, child two_outer_insertion_link, origin xyz=-0.520 0 -0.0155 rpy=0 0 0, axis 0 0 1, mimic joint=two_outer_pitch multiplier=1
- added joint two_outer_roll: type revolute, parent two_tool_main_link, child two_tool_wrist_link, origin xyz=0 0 0.4162 rpy=0 0 0, axis 0 0 1, limit lower=-2.2689 upper=2.2689 effort=1000 velocity=.4
- added joint two_outer_roll_shaft: type fixed, parent two_tool_wrist_link, child two_tool_wrist_shaft_link, origin xyz=0 0 0.0 rpy=0 0 0, axis 0 0 1
- added joint two_outer_yaw: type revolute, parent two_psm_base_link, child two_outer_yaw_link, origin xyz=0.0 0.0 0.0 rpy=0 -1.5708 1.5708, axis 0 0 1, limit lower=-1.5707 upper=1.5707 effort=1000 velocity=.4

File: dvrk_model/model/ecm.urdf.xacro (robot description, xacro)
@@ -41,5 +41,5 @@
     <link name="${prefix}_base_link"/>
     <!-- Joint 1: Outer Yaw -->
-    <joint name="${prefix}_yaw_joint" type="revolute">
+    <joint name="${prefix}_yaw" type="revolute">
       <parent link="${prefix}_base_link"/>
       <child link="${prefix}_yaw_link"/>
@@ -67,5 +67,5 @@
     </link>
     <!-- Joint 2: Pitch -->
-    <joint name="${prefix}_pitch_joint" type="revolute">
+    <joint name="${prefix}_pitch" type="revolute">
       <parent link="${prefix}_yaw_link"/>
       <child link="${prefix}_pitch_link"/>
@@ -76,5 +76,5 @@
     </joint>
     <link name="${prefix}_pitch_link"/>
-    <joint name="${prefix}_pitch_joint_0" type="continuous">
+    <joint name="${prefix}_pitch_0" type="continuous">
       <parent link="${prefix}_yaw_link"/>
       <child link="${prefix}_pitch_link_1"/>
@@ -103,5 +103,5 @@
       </inertial>
     </link>
-    <joint name="${prefix}_pitch_joint_1" type="continuous">
+    <joint name="${prefix}_pitch_1" type="continuous">
       <parent link="${prefix}_pitch_link_1"/>
       <child link="${prefix}_pitch_link_2"/>
@@ -109,5 +109,5 @@
       <axis xyz="0 0 1"/>
       <joint_properties damping="1.0" friction="0.0"/>
-      <mimic joint="${prefix}_pitch_joint" multiplier="-1"/>
+      <mimic joint="${prefix}_pitch" multiplier="-1"/>
     </joint>
     <link name="${prefix}_pitch_link_2">
@@ -130,5 +130,5 @@
       </inertial>
     </link>
-    <joint name="${prefix}_pitch_joint_2" type="continuous">
+    <joint name="${prefix}_pitch_2" type="continuous">
       <parent link="${prefix}_pitch_link_2"/>
       <child link="${prefix}_pitch_link_3"/>
@@ -136,5 +136,5 @@
       <axis xyz="0 0 1"/>
       <joint_properties damping="1.0" friction="0.0"/>
-      <mimic joint="${prefix}_pitch_joint" multiplier="1"/>
+      <mimic joint="${prefix}_pitch" multiplier="1"/>
     </joint>
     <link name="${prefix}_pitch_link_3">
@@ -158,5 +158,5 @@
     </link>
     <!-- Joint 3: Insertion -->
-    <joint name="${prefix}_insertion_joint" type="prismatic">
+    <joint name="${prefix}_insertion" type="prismatic">
       <parent link="${prefix}_pitch_link"/>
       <child link="${prefix}_insertion_link"/>
@@ -182,5 +182,5 @@
     </link>
     <!-- Joint 4: Roll -->
-    <joint name="${prefix}_roll_joint" type="revolute">
+    <joint name="${prefix}_roll" type="revolute">
       <parent link="${prefix}_insertion_link"/>
       <child link="${prefix}_roll_link"/>

File: dvrk_model/model/gazebo_psm.base.urdf.xacro (robot description, xacro)
@@ -29,5 +29,5 @@
     </link>
     <!-- joint 1 -->
-    <joint name="${prefix}outer_yaw_joint" type="revolute">
+    <joint name="${prefix}outer_yaw" type="revolute">
       <parent link="${prefix}psm_base_link"/>
       <child link="${prefix}outer_yaw_link"/>
@@ -59,5 +59,5 @@
     <!-- link, all visual links mimic outer_pitch_joint value -->
     <!-- joint 2: outer_pitch -->
-    <joint name="${prefix}outer_pitch_joint" type="revolute">
+    <joint name="${prefix}outer_pitch" type="revolute">
       <parent link="${prefix}outer_yaw_link"/>
       <child link="${prefix}outer_pitch_link"/>
@@ -80,5 +80,5 @@
     <!--wsn: for visualization links/joints of closed-chain mechanism, assign dynamic properties and control w/ fdbk-->
     <!-- joint 2-1: outer_pitch_1 -->
-    <joint name="${prefix}outer_pitch_joint_1" type="continuous">
+    <joint name="${prefix}outer_pitch_1" type="continuous">
       <parent link="${prefix}outer_yaw_link"/>
       <child link="${prefix}outer_pitch_back_link"/>
@@ -108,5 +108,5 @@
     </link>
     <!-- joint 2-2: outer_pitch_2 -->
-    <joint name="${prefix}outer_pitch_joint_2" type="continuous">
+    <joint name="${prefix}outer_pitch_2" type="continuous">
       <parent link="${prefix}outer_yaw_link"/>
       <child link="${prefix}outer_pitch_front_link"/>
@@ -135,5 +135,5 @@
     </link>
     <!-- joint 2-3: outer_pitch_3 -->
-    <joint name="${prefix}outer_pitch_joint_3" type="continuous">
+    <joint name="${prefix}outer_pitch_3" type="continuous">
       <parent link="${prefix}outer_pitch_back_link"/>
       <child link="${prefix}outer_pitch_bottom_link"/>
@@ -162,5 +162,5 @@
     </link>
     <!-- joint 2-4: outer_pitch_4 -->
-    <joint name="${prefix}outer_pitch_joint_4" type="continuous">
+    <joint name="${prefix}outer_pitch_4" type="continuous">
       <parent link="${prefix}outer_pitch_back_link"/>
       <child link="${prefix}outer_pitch_top_link"/>
@@ -189,5 +189,5 @@
     </link>
     <!-- joint 2-5: outer_pitch_5 -->
-    <joint name="${prefix}outer_pitch_joint_5" type="continuous">
+    <joint name="${prefix}outer_pitch_5" type="continuous">
       <parent link="${prefix}outer_pitch_bottom_link"/>
       <child link="${prefix}outer_insertion_link"/>
@@ -216,5 +216,5 @@
     </link>
     <!-- joint 3: insertion -->
-    <joint name="${prefix}outer_insertion_joint" type="prismatic">
+    <joint name="${prefix}outer_insertion" type="prismatic">
       <!-- <parent link="${prefix}outer_insertion_link"/> -->
       <!-- <parent link="${prefix}psm_base_link"/> -->
@@ -244,5 +244,5 @@
     </link>
     <!-- joint 4: Outer Roll -->
-    <joint name="${prefix}outer_roll_joint" type="revolute">
+    <joint name="${prefix}outer_roll" type="revolute">
       <parent link="${prefix}tool_main_link"/>
       <child link="${prefix}tool_wrist_link"/>
@@ -295,5 +295,5 @@
   <transmission name="${prefix}tran1">
     <type>transmission_interface/SimpleTransmission</type>
-    <joint name="${prefix}outer_yaw_joint">
+    <joint name="${prefix}outer_yaw">
       <hardwareInterface>EffortJointInterface</hardwareInterface>
     </joint>
@@ -305,5 +305,5 @@
   <transmission name="${prefix}tran2">
     <type>transmission_interface/SimpleTransmission</type>
-    <joint name="${prefix}outer_pitch_joint">
+    <joint name="${prefix}outer_pitch">
       <hardwareInterface>EffortJointInterface</hardwareInterface>
     </joint>
@@ -315,5 +315,5 @@
   <transmission name="${prefix}tran2_1">
     <type>transmission_interface/SimpleTransmission</type>
-    <joint name="${prefix}outer_pitch_joint_1">
+    <joint name="${prefix}outer_pitch_1">
       <hardwareInterface>EffortJointInterface</hardwareInterface>
     </joint>
@@ -325,5 +325,5 @@
     <transmission name="${prefix}tran2_2">
     <type>transmission_interface/SimpleTransmission</type>
-    <joint name="${prefix}outer_pitch_joint_2">
+    <joint name="${prefix}outer_pitch_2">
       <hardwareInterface>EffortJointInterface</hardwareInterface>
     </joint>
@@ -335,5 +335,5 @@
       <transmission name="${prefix}tran2_3">
     <type>transmission_interface/SimpleTransmission</type>
-    <joint name="${prefix}outer_pitch_joint_3">
+    <joint name="${prefix}outer_pitch_3">
       <hardwareInterface>EffortJointInterface</hardwareInterface>
     </joint>
@@ -345,5 +345,5 @@
       <transmission name="${prefix}tran2_4">
     <type>transmission_interface/SimpleTransmission</type>
-    <joint name="${prefix}outer_pitch_joint_4">
+    <joint name="${prefix}outer_pitch_4">
       <hardwareInterface>EffortJointInterface</hardwareInterface>
     </joint>
@@ -355,5 +355,5 @@
   <transmission name="${prefix}tran2_5">
     <type>transmission_interface/SimpleTransmission</type>
-    <joint name="${prefix}outer_pitch_joint_5">
+    <joint name="${prefix}outer_pitch_5">
       <hardwareInterface>EffortJointInterface</hardwareInterface>
     </joint>
@@ -365,5 +365,5 @@
   <transmission name="${prefix}tran3">
     <type>transmission_interface/SimpleTransmission</type>
-    <joint name="${prefix}outer_insertion_joint">
+    <joint name="${prefix}outer_insertion">
       <hardwareInterface>EffortJointInterface</hardwareInterface>
     </joint>
@@ -375,5 +375,5 @@
     <transmission name="${prefix}tran4">
     <type>transmission_interface/SimpleTransmission</type>
-    <joint name="${prefix}outer_roll_joint">
+    <joint name="${prefix}outer_roll">
       <hardwareInterface>EffortJointInterface</hardwareInterface>
     </joint>

File: dvrk_model/model/gazebo_psm.tool.sca.urdf.xacro (robot description, xacro)
@@ -8,5 +8,5 @@
   <xacro:macro name="psm_tool_sca" params="prefix">
     <!-- joint 5: Outer wrist pitch joint -->
-    <joint name="${prefix}outer_wrist_pitch_joint" type="revolute">
+    <joint name="${prefix}outer_wrist_pitch" type="revolute">
       <parent link="${prefix}tool_wrist_shaft_link"/>
       <child link="${prefix}tool_wrist_sca_link"/>
@@ -44,5 +44,5 @@
     </link>
     <!-- joint 6: Outer wrist yaw joint -->
-    <joint name="${prefix}outer_wrist_yaw_joint" type="revolute">
+    <joint name="${prefix}outer_wrist_yaw" type="revolute">
       <parent link="${prefix}tool_wrist_sca_link"/>
       <child link="${prefix}tool_wrist_sca_shaft_link"/>
@@ -70,5 +70,5 @@
     </link>
     <!-- joint 7-1: Outer open angle 1  -->
-    <joint name="${prefix}outer_wrist_open_angle_joint" type="revolute">
+    <joint name="${prefix}outer_wrist_open_angle" type="revolute">
       <parent link="${prefix}tool_wrist_sca_shaft_link"/>
       <child link="${prefix}tool_wrist_sca_ee_link_1"/>
@@ -95,5 +95,5 @@
     </link>
     <!-- joint 7-2: Outer open angle 2   -->
-    <joint name="${prefix}outer_wrist_open_angle_joint_mimic" type="revolute">
+    <joint name="${prefix}outer_wrist_open_angle_mimic" type="revolute">
       <parent link="${prefix}tool_wrist_sca_shaft_link"/>
       <child link="${prefix}tool_wrist_sca_ee_link_2"/>
@@ -232,5 +232,5 @@
  <transmission name="${prefix}tran5">
     <type>transmission_interface/SimpleTransmission</type>
-    <joint name="${prefix}outer_wrist_pitch_joint">
+    <joint name="${prefix}outer_wrist_pitch">
       <hardwareInterface>EffortJointInterface</hardwareInterface>
     </joint>
@@ -242,5 +242,5 @@
   <transmission name="${prefix}tran6">
     <type>transmission_interface/SimpleTransmission</type>
-    <joint name="${prefix}outer_wrist_yaw_joint">
+    <joint name="${prefix}outer_wrist_yaw">
       <hardwareInterface>EffortJointInterface</hardwareInterface>
     </joint>
@@ -252,5 +252,5 @@
   <transmission name="${prefix}tran7">
     <type>transmission_interface/SimpleTransmission</type>
-    <joint name="${prefix}outer_wrist_open_angle_joint">
+    <joint name="${prefix}outer_wrist_open_angle">
       <hardwareInterface>EffortJointInterface</hardwareInterface>
     </joint>
@@ -262,5 +262,5 @@
   <transmission name="${prefix}tran7_mimic">
     <type>transmission_interface/SimpleTransmission</type>
-    <joint name="${prefix}outer_wrist_open_angle_joint_mimic">
+    <joint name="${prefix}outer_wrist_open_angle_mimic">
       <hardwareInterface>EffortJointInterface</hardwareInterface>
     </joint>

File: dvrk_model/model/gazebo_psm.tool_w_needle.sca.urdf.xacro (robot description, xacro)
@@ -8,5 +8,5 @@
   <xacro:macro name="psm_tool_sca" params="prefix">
     <!-- joint 5: Outer wrist pitch joint -->
-    <joint name="${prefix}outer_wrist_pitch_joint" type="revolute">
+    <joint name="${prefix}outer_wrist_pitch" type="revolute">
       <parent link="${prefix}tool_wrist_shaft_link"/>
       <child link="${prefix}tool_wrist_sca_link"/>
@@ -44,5 +44,5 @@
     </link>
     <!-- joint 6: Outer wrist yaw joint -->
-    <joint name="${prefix}outer_wrist_yaw_joint" type="revolute">
+    <joint name="${prefix}outer_wrist_yaw" type="revolute">
       <parent link="${prefix}tool_wrist_sca_link"/>
       <child link="${prefix}tool_wrist_sca_shaft_link"/>
@@ -70,5 +70,5 @@
     </link>
     <!-- joint 7-1: Outer open angle 1  -->
-    <joint name="${prefix}outer_wrist_open_angle_joint" type="revolute">
+    <joint name="${prefix}outer_wrist_open_angle" type="revolute">
       <parent link="${prefix}tool_wrist_sca_shaft_link"/>
       <child link="${prefix}tool_wrist_sca_ee_link_1"/>
@@ -95,5 +95,5 @@
     </link>
     <!-- joint 7-2: Outer open angle 2   -->
-    <joint name="${prefix}outer_wrist_open_angle_joint_mimic" type="revolute">
+    <joint name="${prefix}outer_wrist_open_angle_mimic" type="revolute">
       <parent link="${prefix}tool_wrist_sca_shaft_link"/>
       <child link="${prefix}tool_wrist_sca_ee_link_2"/>
@@ -257,5 +257,5 @@
  <transmission name="${prefix}tran5">
     <type>transmission_interface/SimpleTransmission</type>
-    <joint name="${prefix}outer_wrist_pitch_joint">
+    <joint name="${prefix}outer_wrist_pitch">
       <hardwareInterface>EffortJointInterface</hardwareInterface>
     </joint>
@@ -267,5 +267,5 @@
   <transmission name="${prefix}tran6">
     <type>transmission_interface/SimpleTransmission</type>
-    <joint name="${prefix}outer_wrist_yaw_joint">
+    <joint name="${prefix}outer_wrist_yaw">
       <hardwareInterface>EffortJointInterface</hardwareInterface>
     </joint>
@@ -277,5 +277,5 @@
   <transmission name="${prefix}tran7">
     <type>transmission_interface/SimpleTransmission</type>
-    <joint name="${prefix}outer_wrist_open_angle_joint">
+    <joint name="${prefix}outer_wrist_open_angle">
       <hardwareInterface>EffortJointInterface</hardwareInterface>
     </joint>
@@ -287,5 +287,5 @@
   <transmission name="${prefix}tran7_mimic">
     <type>transmission_interface/SimpleTransmission</type>
-    <joint name="${prefix}outer_wrist_open_angle_joint_mimic">
+    <joint name="${prefix}outer_wrist_open_angle_mimic">
       <hardwareInterface>EffortJointInterface</hardwareInterface>
     </joint>
