Commit message: Made the DaVinci arms color coded to match the real arms.

File: davinci_gazebo/model/both_psms_sticky.urdf.xacro (robot description, xacro)
@@ -54,6 +54,6 @@
 		<!--origin rpy="0.0 0.0 0.0" xyz="0.0 0.2 0.8"/-->
 	</link>
-	<xacro:psm_sca prefix="one_" parent_link="camera" xyz="-0.15 0.05 0.5" rpy="0.0 0.0 3.1415926"/>
-	<xacro:psm_sca prefix="two_" parent_link="camera" xyz="0.15 0.05 0.5" rpy="0.0 0.0 3.1415926"/>
+	<xacro:psm_sca prefix="two_" colorcode="Green" parent_link="camera" xyz="-0.15 0.05 0.5" rpy="0.0 0.0 3.1415926"/>
+	<xacro:psm_sca prefix="one_" colorcode="Yellow" parent_link="camera" xyz="0.15 0.05 0.5" rpy="0.0 0.0 3.1415926"/>
 	<!-- ros_control plugin -->
 	<gazebo>

File: davinci_gazebo/model/gazebo_psm_sticky.tool.sca.urdf.xacro (robot description, xacro)
@@ -209,5 +209,5 @@
 			</visual>
 		</link>
-		<!--this colors the tool-tip fiducial red; oddly, this shows up in the camera view, but NOT in the rviz view -->
+		<!--this colors the tool-tip fiducial; oddly, this shows up in the camera view, but NOT in the rviz view -->
 		<gazebo reference="${prefix}tool_tip_link">
 			<material>Gazebo/Red</material>

File: davinci_gazebo/model/psm_sticky.urdf.xacro (robot description, xacro)
@@ -2,11 +2,12 @@
 <robot name="dvrk_psm" xmlns:xacro="http://www.ros.org/wiki/xacro">
   <!-- Macros -->
-  <xacro:include filename="$(find dvrk_model)/model/gazebo_psm.base.urdf.xacro"/>
+  <xacro:include filename="$(find davinci_gazebo)/model/gazebo_psm.base.urdf.xacro"/>
   <xacro:include filename="$(find davinci_gazebo)/model/gazebo_psm_sticky.tool.sca.urdf.xacro"/>
   <!--xacro:include filename="$(find dvrk_model)/model/psm.tool.caudier.urdf.xacro"/-->
   <!-- Macro for psm with sca -->
-  <xacro:macro name="psm_sca" params="prefix parent_link xyz rpy">
+  <xacro:macro name="psm_sca" params="prefix colorcode parent_link xyz rpy">
     <xacro:psm
         prefix="${prefix}"
+        colorcode="${colorcode}"
         parent_link="${parent_link}"
         xyz="${xyz}" rpy="${rpy}"/>
