Commit message: Ascended the interface and trajectory interpolator; removed some outdated packages of unknown purpose (you can still find them in the main repository).

File: davinci_gazebo/model/gazebo_psm.base.urdf.xacro (robot description, xacro)
@@ -16,5 +16,5 @@
         <origin rpy="1.5708 0 3.1416" xyz="0.039 -0.40788 -0.07879"/>
         <geometry>
-          <mesh filename="package://dvrk_model/meshes/psm/psm_base.dae"/>
+          <mesh filename="package://davinci_gazebo/meshes/psm/psm_base.dae"/>
         </geometry>
       </visual>
@@ -43,5 +43,5 @@
         <origin rpy="3.1416 0 1.5708" xyz="0.0125 0 0.5265"/>
         <geometry>
-          <mesh filename="package://dvrk_model/meshes/psm/outer_yaw.dae"/>
+          <mesh filename="package://davinci_gazebo/meshes/psm/outer_yaw.dae"/>
         </geometry>
       </visual>
@@ -95,5 +95,5 @@
         <origin rpy="0 0 -0.27129" xyz="0 0 0"/>
         <geometry>
-          <mesh filename="package://dvrk_model/meshes/psm/outer_pitch_back.dae"/>
+          <mesh filename="package://davinci_gazebo/meshes/psm/outer_pitch_back.dae"/>
         </geometry>
       </visual>
@@ -122,5 +122,5 @@
         <origin rpy="0 0 -0.27129" xyz="0 0 0"/>
         <geometry>
-          <mesh filename="package://dvrk_model/meshes/psm/outer_pitch_front.dae"/>
+          <mesh filename="package://davinci_gazebo/meshes/psm/outer_pitch_front.dae"/>
         </geometry>
       </visual>
@@ -149,5 +149,5 @@
         <origin rpy="0 -1.5708 0" xyz="0.009 0 0"/>
         <geometry>
-          <mesh filename="package://dvrk_model/meshes/psm/outer_pitch_bottom.dae"/>
+          <mesh filename="package://davinci_gazebo/meshes/psm/outer_pitch_bottom.dae"/>
         </geometry>
       </visual>
@@ -176,5 +176,5 @@
         <origin rpy="0 -1.5708 0" xyz="0.009 0 0"/>
         <geometry>
-          <mesh filename="package://dvrk_model/meshes/psm/outer_pitch_top.dae"/>
+          <mesh filename="package://davinci_gazebo/meshes/psm/outer_pitch_top.dae"/>
         </geometry>
       </visual>
@@ -203,5 +203,5 @@
         <origin rpy="0 -1.5708 1.5708" xyz="0.02528 0.429 0"/>
         <geometry>
-          <mesh filename="package://dvrk_model/meshes/psm/outer_insertion.dae"/>
+          <mesh filename="package://davinci_gazebo/meshes/psm/outer_insertion.dae"/>
         </geometry>
       </visual>
@@ -234,5 +234,5 @@
         <origin rpy="0 0 1.5708" xyz="0 0 0.041"/>
         <geometry>
-          <mesh filename="package://dvrk_model/meshes/psm/tool_main.dae"/>
+          <mesh filename="package://davinci_gazebo/meshes/psm/tool_main.dae"/>
         </geometry>
       </visual>
@@ -260,5 +260,5 @@
         <origin rpy="0 0 1.5708" xyz="0 0 -0.0091"/>
         <geometry>
-          <mesh filename="package://dvrk_model/meshes/psm/tool_wrist_link.dae"/>
+          <mesh filename="package://davinci_gazebo/meshes/psm/tool_wrist_link.dae"/>
         </geometry>
       </visual>
@@ -284,5 +284,5 @@
         <origin rpy="1.5708 0 0" xyz="0 0.00401 0"/>
         <geometry>
-          <mesh filename="package://dvrk_model/meshes/psm/tool_wrist_shaft_link.dae"/>
+          <mesh filename="package://davinci_gazebo/meshes/psm/tool_wrist_shaft_link.dae"/>
         </geometry>
       </visual>

File: davinci_gazebo/model/gazebo_psm_sticky.tool.sca.urdf.xacro (robot description, xacro)
@@ -2,5 +2,5 @@
 <robot name="dvrk_psm" xmlns:xacro="http://www.ros.org/wiki/xacro">
 	<!-- This file contains different tool urdf -->
-	<xacro:include filename="$(find dvrk_model)/model/common.urdf.xacro"/>
+	<xacro:include filename="$(find davinci_gazebo)/model/common.urdf.xacro"/>
 	<!-- TOM: pretty sure this does not actually, if you want to get technical about it, DO anything.-->
 	<!--xacro:property name="GazeboRed"       value="1 0 0 1"/>
@@ -23,5 +23,5 @@
 				<origin rpy="1.5708 3.1416 0" xyz="0.0051 0.0032 0"/>
 				<geometry>
-					<mesh filename="package://dvrk_model/meshes/psm/tool_wrist_sca_link.dae"/>
+					<mesh filename="package://davinci_gazebo/meshes/psm/tool_wrist_sca_link.dae"/>
 				</geometry>
 			</visual>
@@ -31,5 +31,5 @@
 					<!-- coarse model; a simple box -->
 					<!--box size="0.05 0.2 0.05"/-->
-					<mesh filename="package://dvrk_model/meshes/psm/tool_wrist_sca_link.dae"/>
+					<mesh filename="package://davinci_gazebo/meshes/psm/tool_wrist_sca_link.dae"/>
 				</geometry>
 			</collision>
@@ -55,5 +55,5 @@
 				<origin rpy="0 0 0" xyz="0 -0.0002 -0.0025"/>
 				<geometry>
-					<mesh filename="package://dvrk_model/meshes/psm/tool_wrist_sca_shaft_link.dae"/>
+					<mesh filename="package://davinci_gazebo/meshes/psm/tool_wrist_sca_shaft_link.dae"/>
 				</geometry>
 			</visual>
@@ -77,5 +77,5 @@
 				<origin rpy="0 0 0" xyz="0 0 0"/>
 				<geometry>
-					<mesh filename="package://dvrk_model/meshes/psm/tool_wrist_sca_link_2.dae"/>
+					<mesh filename="package://davinci_gazebo/meshes/psm/tool_wrist_sca_link_2.dae"/>
 				</geometry>
 			</visual>
@@ -100,5 +100,5 @@
 				<origin rpy="0 3.1516 0" xyz="0 0 0"/>
 				<geometry>
-					<mesh filename="package://dvrk_model/meshes/psm/tool_wrist_sca_link_2.dae"/>
+					<mesh filename="package://davinci_gazebo/meshes/psm/tool_wrist_sca_link_2.dae"/>
 				</geometry>
 			</visual>
